File: kicadFiles/muente1800.kicad_pcb (KiCad board)
At the start: 2 copper layers, 162 parts, among them SW1 MXSwitch_100, SW10 MXSwitch_100, SW11 MXSwitch_100, SW12 MXSwitch_100, SW13 MXSwitch_100, SW14 MXSwitch_200, SW15 MXSwitch_100, SW16 MXSwitch_100, SW17 MXSwitch_100, SW18 MXSwitch_100, SW19 MXSwitch_150, SW2 MXSwitch_100, SW20 MXSwitch_100, SW21 MXSwitch_100, SW22 MXSwitch_100, SW23 MXSwitch_100, SW24 MXSwitch_100, SW25 MXSwitch_100, SW26 MXSwitch_100, SW27 MXSwitch_100, SW28 MXSwitch_100, SW29 MXSwitch_100, SW3 MXSwitch_100, SW30 MXSwitch_100, SW31 MXSwitch_100, SW32 MXSwitch_100, SW33 MXSwitch_100, SW34 MXSwitch_100, SW35 MXSwitch_175, SW36 MXSwitch_100, SW37 MXSwitch_100, SW38 MXSwitch_100, SW39 MXSwitch_100, SW4 MXSwitch_100, SW40 MXSwitch_100, SW41 MXSwitch_100, SW42 MXSwitch_100, SW43 MXSwitch_100, SW44 MXSwitch_100, SW45 MXSwitch_100, SW46 MXSwitch_100, SW47 MXSwitch_100, SW48 MXSwitch_ISO, SW49 MXSwitch_100, SW5 MXSwitch_100, SW50 MXSwitch_100, SW51 MXSwitch_100, SW52 MXSwitch_200, SW53 MXSwitch_125, SW54 MXSwitch_100, SW55 MXSwitch_100, SW56 MXSwitch_100, SW57 MXSwitch_100, SW58 MXSwitch_100, SW59 MXSwitch_100, SW6 MXSwitch_100, SW60 MXSwitch_100, SW61 MXSwitch_100, SW62 MXSwitch_100, SW63 MXSwitch_100, SW64 MXSwitch_100, SW65 MXSwitch_175, SW66 MXSwitch_100, SW67 MXSwitch_100, SW68 MXSwitch_100, SW69 MXSwitch_100, SW7 MXSwitch_100, SW70 MXSwitch_125, SW71 MXSwitch_125, SW72 MXSwitch_125, SW73 MXSwitch_625, SW74 MXSwitch_150, SW75 MXSwitch_150, SW76 MXSwitch_100, SW77 MXSwitch_100, SW78 MXSwitch_100, SW79 MXSwitch_100, SW8 MXSwitch_100, SW80 MXSwitch_100, SW81 MXSwitch_200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

Commit message: edge cut
Parts:
- added REF**: 60_Outline, 60_Outline-Modded, F.Cu at (176.2, 38.1)
Other:
- board outline added: 370.7 x 95.1 mm
Changed lines of the file:
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@@
     (tracks 0)
     (zones 0)
-    (modules 162)
+    (modules 163)
     (nets 105)
   )
@@
     (add_net row4)
   )
+  (module 60_Outline-Modded (layer F.Cu)
+    (at 176.2125 38.1)
+    (fp_text reference REF** (at -181.865 50.5) (layer Edge.Cuts) hide
+      (effects (font (size 1 1) (thickness 0.15)))
+    )
+    (fp_text value 60_Outline (at -181.865 49) (layer F.Fab) hide
+      (effects (font (size 1 1) (thickness 0.15)))
+    )
+    (fp_line (start -183.365 47.3) (end 183.365 47.3) (layer Edge.Cuts) (width 0.3))
+    (fp_line (start 183.365 -47.3) (end -161.165 -47.3) (layer Edge.Cuts) (width 0.3))
+    (fp_arc (start -183.365 -45.3) (end -185.365 -45.3) (angle 90) (layer Edge.Cuts) (width 0.3))
+    (fp_arc (start -183.365 45.3) (end -183.365 47.3) (angle 90) (layer Edge.Cuts) (width 0.3))
+    (fp_arc (start 183.365 45.3) (end 185.365 45.3) (angle 90) (layer Edge.Cuts) (width 0.3))
+    (fp_arc (start 183.365 -45.3) (end 183.365 -47.3) (angle 90) (layer Edge.Cuts) (width 0.3))
+    (fp_line (start -185.365 45.3) (end -185.365 10.6) (layer Edge.Cuts) (width 0.3))
+    (fp_line (start -185.365 10.6) (end -181.565 10.6) (layer Edge.Cuts) (width 0.3))
+    (fp_arc (start -181.565 9.2) (end -181.565 7.8) (angle 90) (layer Edge.Cuts) (width 0.3))
+    (fp_line (start -181.565 7.8) (end -185.365 7.8) (layer Edge.Cuts) (width 0.3))
+    (fp_line (start -185.365 7.8) (end -185.365 -45.3) (layer Edge.Cuts) (width 0.3))
+    (fp_arc (start 181.565 9.2) (end 181.565 7.8) (angle -90) (layer Edge.Cuts) (width 0.3))
+    (fp_arc (start 181.565 9.2) (end 180.165 9.2) (angle -90) (layer Edge.Cuts) (width 0.3))
+    (fp_line (start 185.365 10.6) (end 185.365 45.3) (layer Edge.Cuts) (width 0.3))
+    (fp_line (start 185.365 7.8) (end 185.365 -45.3) (layer Edge.Cuts) (width 0.3))
+    (fp_line (start 181.565 10.6) (end 185.365 10.6) (layer Edge.Cuts) (width 0.3))
+    (fp_line (start 181.565 7.8) (end 185.365 7.8) (layer Edge.Cuts) (width 0.3))
+    (fp_line (start -185.365 6.54905) (end -181.565 6.54905) (layer F.Cu) (width 2.5019))
+    (fp_line (start -185.365 6.54905) (end -181.565 6.54905) (layer B.Cu) (width 2.5019))
+    (fp_arc (start -181.565 9.2) (end -180.165 9.2) (angle 90) (layer Edge.Cuts) (width 0.3))
+    (fp_arc (start -181.565 9.2) (end -178.91405 9.2) (angle 90) (layer F.Cu) (width 2.5019))
+    (fp_arc (start -181.565 9.2) (end -181.565 6.54905) (angle 90) (layer F.Cu) (width 2.5019))
+    (fp_line (start -185.365 11.85095) (end -181.565 11.85095) (layer B.Cu) (width 2.5019))
+    (fp_line (start -185.365 11.85095) (end -181.565 11.85095) (layer F.Cu) (width 2.5019))
+    (fp_arc (start -181.565 9.2) (end -178.91405 9.2) (angle 90) (layer B.Cu) (width 2.5019))
+    (fp_arc (start -181.565 9.2) (end -181.565 6.54905) (angle 90) (layer B.Cu) (width 2.5019))
+    (fp_arc (start 181.565 9.2) (end 181.565 6.54905) (angle -90) (layer B.Cu) (width 2.5019))
+    (fp_arc (start 181.565 9.2) (end 178.91405 9.2) (angle -90) (layer B.Cu) (width 2.5019))
+    (fp_line (start 181.565 11.85095) (end 185.415 11.85095) (layer F.Cu) (width 2.5019))
+    (fp_line (start 181.565 6.54905) (end 185.365 6.54905) (layer B.Cu) (width 2.5019))
+    (fp_arc (start 181.565 9.2) (end 181.565 6.54905) (angle -90) (layer F.Cu) (width 2.5019))
+    (fp_arc (start 181.565 9.2) (end 178.91405 9.2) (angle -90) (layer F.Cu) (width 2.5019))
+    (fp_line (start 181.565 6.54905) (end 185.365 6.54905) (layer F.Cu) (width 2.5019))
+    (fp_line (start 181.565 11.85095) (end 185.415 11.85095) (layer B.Cu) (width 2.5019))
+    (fp_line (start -185.365 11.85095) (end -181.565 11.85095) (layer F.Mask) (width 2.5019))
+    (fp_line (start -185.365 11.85095) (end -181.565 11.85095) (layer B.Mask) (width 2.5019))
+    (fp_arc (start -181.565 9.2) (end -178.91405 9.2) (angle 90) (layer B.Mask) (width 2.5019))
+    (fp_arc (start -181.565 9.2) (end -178.91405 9.2) (angle 90) (layer F.Mask) (width 2.5019))
+    (fp_arc (start -181.565 9.2) (end -181.565 6.54905) (angle 90) (layer F.Mask) (width 2.5019))
+    (fp_arc (start -181.565 9.2) (end -181.565 6.54905) (angle 90) (layer B.Mask) (width 2.5019))
+    (fp_line (start -185.365 6.54905) (end -181.565 6.54905) (layer F.Mask) (width 2.5019))
+    (fp_line (start -185.365 6.54905) (end -181.565 6.54905) (layer B.Mask) (width 2.5019))
+    (fp_line (start 181.565 11.85095) (end 185.415 11.85095) (layer B.Mask) (width 2.5019))
+    (fp_line (start 181.565 11.85095) (end 185.415 11.85095) (layer F.Mask) (width 2.5019))
+    (fp_arc (start 181.565 9.2) (end 178.91405 9.2) (angle -90) (layer F.Mask) (width 2.5019))
+    (fp_arc (start 181.565 9.2) (end 178.91405 9.2) (angle -90) (layer B.Mask) (width 2.5019))
+    (fp_arc (start 181.565 9.2) (end 181.565 6.54905) (angle -90) (layer F.Mask) (width 2.5019))
+    (fp_arc (start 181.565 9.2) (end 181.565 6.54905) (angle -90) (layer B.Mask) (width 2.5019))
+    (fp_line (start 181.565 6.54905) (end 185.365 6.54905) (layer B.Mask) (width 2.5019))
+    (fp_line (start 181.565 6.54905) (end 185.365 6.54905) (layer F.Mask) (width 2.5019))
+    (fp_line (start -172.665 -47.8) (end -161.665 -47.8) (layer Edge.Cuts) (width 0.3))
+    (fp_arc (start -173.165 -47.8) (end -172.665 -47.8) (angle 90) (layer Edge.Cuts) (width 0.3))
+    (fp_arc (start -161.165 -47.8) (end -161.165 -47.3) (angle 90) (layer Edge.Cuts) (width 0.3))
+    (fp_line (start -183.365 -47.3) (end -173.165 -47.3) (layer Edge.Cuts) (width 0.3))
+    (fp_line (start -167.165 -48.9) (end -167.165 -45.75) (layer Dwgs.User) (width 0.15))
+    (pad 1 thru_hole circle (at 179.726522 11.038478) (size 1 1) (drill 0.5) (layers *.Cu *.Mask))
+    (pad 1 thru_hole circle (at 181.565 11.8) (size 1 1) (drill 0.5) (layers *.Cu *.Mask))
+    (pad 1 thru_hole circle (at 183.607035 11.8) (size 1 1) (drill 0.5) (layers *.Cu *.Mask))
+    (pad 1 thru_hole circle (at 183.607035 6.6) (size 1 1) (drill 0.5) (layers *.Cu *.Mask))
+    (pad 1 thru_hole circle (at 181.565 6.6) (size 1 1) (drill 0.5) (layers *.Cu *.Mask))
+    (pad 1 thru_hole circle (at 179.726522 7.361522) (size 1 1) (drill 0.5) (layers *.Cu *.Mask))
+    (pad 1 thru_hole circle (at 178.965 9.2) (size 1 1) (drill 0.5) (layers *.Cu *.Mask))
+    (pad 1 thru_hole circle (at -183.607035 11.8) (size 1 1) (drill 0.5) (layers *.Cu *.Mask))
+    (pad 1 thru_hole circle (at -183.607035 6.6) (size 1 1) (drill 0.5) (layers *.Cu *.Mask))
+    (pad 1 thru_hole circle (at -179.726522 11.038478) (size 1 1) (drill 0.5) (layers *.Cu *.Mask))
+    (pad 1 thru_hole circle (at -179.726522 7.361522) (size 1 1) (drill 0.5) (layers *.Cu *.Mask))
+    (pad 1 thru_hole circle (at -181.565 11.8) (size 1 1) (drill 0.5) (layers *.Cu *.Mask))
+    (pad 1 thru_hole circle (at -181.565 6.6) (size 1 1) (drill 0.5) (layers *.Cu *.Mask))
+    (pad 1 thru_hole circle (at -178.965 9.2) (size 1 1) (drill 0.5) (layers *.Cu *.Mask))
+    (pad 1 thru_hole circle (at -55.965 2) (size 1 1) (drill 0.5) (layers *.Cu *.Mask))
+    (pad 1 thru_hole circle (at -58.365 2) (size 1 1) (drill 0.5) (layers *.Cu *.Mask))
+    (pad 1 thru_hole circle (at -57.165 2) (size 1 1) (drill 0.5) (layers *.Cu *.Mask))
+    (pad 1 thru_hole circle (at -58.365 -2.6) (size 1 1) (drill 0.5) (layers *.Cu *.Mask))
+    (pad 1 thru_hole circle (at -55.965 -2.6) (size 1 1) (drill 0.5) (layers *.Cu *.Mask))
+    (pad 1 thru_hole circle (at -57.165 -2.6) (size 1 1) (drill 0.5) (layers *.Cu *.Mask))
+    (pad 1 thru_hole circle (at 6.335 40.2) (size 1 1) (drill 0.5) (layers *.Cu *.Mask))
+    (pad 1 thru_hole circle (at 3.935 40.2) (size 1 1) (drill 0.5) (layers *.Cu *.Mask))
+    (pad 1 thru_hole circle (at 3.935 35.6) (size 1 1) (drill 0.5) (layers *.Cu *.Mask))
+    (pad 1 thru_hole circle (at 6.335 35.6) (size 1 1) (drill 0.5) (layers *.Cu *.Mask))
+    (pad 1 thru_hole circle (at 5.135 40.2) (size 1 1) (drill 0.5) (layers *.Cu *.Mask))
+    (pad 1 thru_hole circle (at 5.135 35.6) (size 1 1) (drill 0.5) (layers *.Cu *.Mask))
+    (pad 1 thru_hole circle (at 75.885 -21.717) (size 1 1) (drill 0.5) (layers *.Cu *.Mask))
+    (pad 1 thru_hole circle (at 73.485 -21.7) (size 1 1) (drill 0.5) (layers *.Cu *.Mask))
+    (pad 1 thru_hole circle (at 73.485 -17.1) (size 1 1) (drill 0.5) (layers *.Cu *.Mask))
+    (pad 1 thru_hole circle (at 75.885 -17.1) (size 1 1) (drill 0.5) (layers *.Cu *.Mask))
+    (pad 1 thru_hole circle (at 74.685 -17.1) (size 1 1) (drill 0.5) (layers *.Cu *.Mask))
+    (pad 1 thru_hole circle (at 74.685 -21.7) (size 1 1) (drill 0.5) (layers *.Cu *.Mask))
+    (pad 1 thru_hole circle (at -158.538654 -17.773654) (size 1 1) (drill 0.5) (layers *.Cu *.Mask))
+    (pad 1 thru_hole circle (at -161.791346 -17.773654) (size 1 1) (drill 0.5) (layers *.Cu *.Mask))
+    (pad 1 thru_hole circle (at -158.538654 -21.026346) (size 1 1) (drill 0.5) (layers *.Cu *.Mask))
+    (pad 1 thru_hole circle (at -161.791346 -21.026346) (size 1 1) (drill 0.5) (layers *.Cu *.Mask))
+    (pad 1 thru_hole circle (at -160.165 -17.1) (size 1 1) (drill 0.5) (layers *.Cu *.Mask))
+    (pad 1 thru_hole circle (at -157.865 -19.4) (size 1 1) (drill 0.5) (layers *.Cu *.Mask))
+    (pad 1 thru_hole circle (at -162.465 -19.4) (size 1 1) (drill 0.5) (layers *.Cu *.Mask))
+    (pad 1 thru_hole circle (at -160.165 -21.7) (size 1 1) (drill 0.5) (layers *.Cu *.Mask))
+    (pad 1 thru_hole circle (at 74.685 -19.4) (size 7.00024 7.00024) (drill oval 5.00126 2.49936) (layers *.Cu *.Mask))
+    (pad 1 thru_hole circle (at 5.135 37.9) (size 7.00024 7.00024) (drill oval 5.00126 2.49936) (layers *.Cu *.Mask))
+    (pad 1 thru_hole circle (at -57.165 -0.3) (size 7.00024 7.00024) (drill oval 5.00126 2.49936) (layers *.Cu *.Mask))
+    (pad 1 thru_hole circle (at -160.165 -19.4) (size 7.0013 7.0013) (drill 2.4994) (layers *.Cu *.Mask))
+  )
   (module acheron_MX:MX200R (layer B.Cu)
