File: kicadFiles/muente1800.kicad_pcb (KiCad board)
At the start: 2 copper layers, 370.7 x 99.9 mm, 163 parts, among them SW1 MXSwitch_100, SW10 MXSwitch_100, SW11 MXSwitch_100, SW12 MXSwitch_100, SW13 MXSwitch_100, SW14 MXSwitch_200, SW15 MXSwitch_100, SW16 MXSwitch_100, SW17 MXSwitch_100, SW18 MXSwitch_100, SW19 MXSwitch_150, SW2 MXSwitch_100, SW20 MXSwitch_100, SW21 MXSwitch_100, SW22 MXSwitch_100, SW23 MXSwitch_100, SW24 MXSwitch_100, SW25 MXSwitch_100, SW26 MXSwitch_100, SW27 MXSwitch_100, SW28 MXSwitch_100, SW29 MXSwitch_100, SW3 MXSwitch_100, SW30 MXSwitch_100, SW31 MXSwitch_100, SW32 MXSwitch_100, SW33 MXSwitch_100, SW34 MXSwitch_100, SW35 MXSwitch_175, SW36 MXSwitch_100, SW37 MXSwitch_100, SW38 MXSwitch_100, SW39 MXSwitch_100, SW4 MXSwitch_100, SW40 MXSwitch_100, SW41 MXSwitch_100, SW42 MXSwitch_100, SW43 MXSwitch_100, SW44 MXSwitch_100, SW45 MXSwitch_100, SW46 MXSwitch_100, SW47 MXSwitch_100, SW48 MXSwitch_ISO, SW49 MXSwitch_100, SW5 MXSwitch_100, SW50 MXSwitch_100, SW51 MXSwitch_100, SW52 MXSwitch_200, SW53 MXSwitch_125, SW54 MXSwitch_100, SW55 MXSwitch_100, SW56 MXSwitch_100, SW57 MXSwitch_100, SW58 MXSwitch_100, SW59 MXSwitch_100, SW6 MXSwitch_100, SW60 MXSwitch_100, SW61 MXSwitch_100, SW62 MXSwitch_100, SW63 MXSwitch_100, SW64 MXSwitch_100, SW65 MXSwitch_175, SW66 MXSwitch_100, SW67 MXSwitch_100, SW68 MXSwitch_100, SW69 MXSwitch_100, SW7 MXSwitch_100, SW70 MXSwitch_125, SW71 MXSwitch_125, SW72 MXSwitch_125, SW73 MXSwitch_625, SW74 MXSwitch_150, SW75 MXSwitch_150, SW76 MXSwitch_100, SW77 MXSwitch_100, SW78 MXSwitch_100, SW79 MXSwitch_100, SW8 MXSwitch_100, SW80 MXSwitch_100, SW81 MXSwitch_200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

Commit message: ground fill
Parts:
- added J1: TYPE-C-31-M12_13, acheron_Connectors:TYPE-C-31-M-12, B.Cu at (9.09, -2.80)
- added U1: STM32F072CBTx, acheron_Components:LQFP-48_7x7mm_P0.5mm, B.Cu at (21.4, 109.5)
- D1, D10, D11, D12, D13, D14, D15, D16, D17, D18, D19, D2, D20, D21, D22, D23, D24, D25, D26, D27, D28, D29, D3, D30, D31, D32, D33, D34, D35, D36, D37, D38, D39, D4, D40, D41, D42, D43, D44, D45, D46, D47, D48, D49, D5, D50, D51, D52, D53, D54, D55, D56, D57, D58, D59, D6, D60, D61, D62, D63, D64, D65, D66, D67, D68, D69, D7, D70, D71, D72, D73, D74, D75, D76, D77, D78, D79, D8, D80, D81, D9: moved to B.Cu
- SW52, SW81: footprint acheron_MX:MX200R -> acheron_MX:MX200
- moved D61 147.0 mm to (146.1, 117.7), turned to 180 degrees
- moved D70 147.0 mm to (146.1, 114.3), turned to 180 degrees
- moved D77 147.0 mm to (146.1, 107.6), turned to 180 degrees
- moved D80 147.0 mm to (146.1, 111.0), turned to 180 degrees
- moved D60 135.3 mm to (140.3, 117.7), turned to 180 degrees
- moved D69 135.3 mm to (140.3, 114.3), turned to 180 degrees
- moved D71 135.3 mm to (140.3, 111.0), turned to 180 degrees
- moved D81 135.3 mm to (140.3, 107.6), turned to 180 degrees
- moved D59 123.6 mm to (134.4, 117.7), turned to 180 degrees
- moved D65 123.6 mm to (134.4, 111.0), turned to 180 degrees
- moved D68 123.6 mm to (134.4, 107.6), turned to 180 degrees
- moved D72 123.6 mm to (134.4, 114.3), turned to 180 degrees
- moved D1 111.9 mm to (128.6, 114.3), turned to 180 degrees
- moved D52 111.9 mm to (128.6, 117.7), turned to 180 degrees
- moved D64 111.9 mm to (128.6, 111.0), turned to 180 degrees
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Routing:
- added copper zone on B.Cu, net GND
- added copper zone on F.Cu, net GND

Commit message: 3d
Parts:
- added C1: 100nF, Capacitor_SMD:C_0805_2012Metric_Pad1.15x1.40mm_HandSolder, B.Cu at (41.3, 7.94)
- added C2: 10uF, Capacitor_SMD:C_0805_2012Metric_Pad1.15x1.40mm_HandSolder, B.Cu at (37.3, 21.4)
- added CB1: 100nF, Capacitor_SMD:C_0805_2012Metric_Pad1.15x1.40mm_HandSolder, B.Cu at (15.9, 38.9)
- added CB2: 100nF, Capacitor_SMD:C_0805_2012Metric_Pad1.15x1.40mm_HandSolder, B.Cu at (11.9, 27.0)
- added CB3: 100nF, Capacitor_SMD:C_0805_2012Metric_Pad1.15x1.40mm_HandSolder, B.Cu at (27.0, 26.2)
- added CB4: 100nF, Capacitor_SMD:C_0805_2012Metric_Pad1.15x1.40mm_HandSolder, B.Cu at (29.4, 31.0)
- added CB5: 10nF, Capacitor_SMD:C_0805_2012Metric_Pad1.15x1.40mm_HandSolder, B.Cu at (27.0, 31.0)
- added CRST1: 4.7nF, Capacitor_SMD:C_0805_2012Metric_Pad1.15x1.40mm_HandSolder, B.Cu at (44.5, 65.1)
- added CRST2: 10uF, Capacitor_SMD:C_0805_2012Metric_Pad1.15x1.40mm_HandSolder, B.Cu at (33.3, 50.8)
- added DRST1: 1N4148, acheron_Components:D_SOD-123, B.Cu at (33.3, 53.3)
- added J2: Conn_ARM_JTAG_SWD_10, acheron_Connectors:Conn_ARM_JTAG_SWD_10, B.Cu at (-4.76, 28.6)
- added QRST1: DTC123J, Package_TO_SOT_SMD:SOT-23_Handsoldering, B.Cu at (39.7, 64.3)
- added R1: 5.1k, Resistor_SMD:R_0805_2012Metric_Pad1.15x1.40mm_HandSolder, B.Cu at (5.71, 3.74)
- added R2: 5.1k, Resistor_SMD:R_0805_2012Metric_Pad1.15x1.40mm_HandSolder, B.Cu at (13.5, 3.97)
- added RRST1: 100k, Resistor_SMD:R_0805_2012Metric_Pad1.15x1.40mm_HandSolder, B.Cu at (33.3, 56.0)
- added SWRST1: SW_Push, acheron_Hardware:K2-1187SQ-A4SW-06, B.Cu at (33.3, 61.9)
- added U2: LD1117S33TR_SOT223, Package_TO_SOT_SMD:SOT-223-3_TabPin2, B.Cu at (38.1, 14.3)
- SW52, SW81: footprint acheron_MX:MX200 -> acheron_MX:MX200R
- SW73: footprint acheron_MX:MX625 -> acheron_MX:MX625R
- moved D18 287.8 mm to (349.2, 4.76), turned to 90 degrees
- moved D17 274.3 mm to (330.2, 4.76), turned to 90 degrees
- moved D33 272.7 mm to (307.2, 13.5), turned to 270 degrees
- moved D79 269.7 mm to (307.2, 70.6), turned to 270 degrees
- moved D16 257.9 mm to (311.1, 4.76), turned to 90 degrees
- moved D78 244.9 mm to (283.4, 75.4), turned to 270 degrees
- moved D15 244.9 mm to (292.1, 4.76), turned to 90 degrees
- moved D34 244.4 mm to (326.2, 13.5), turned to 270 degrees
- moved D32 229.0 mm to (288.1, 13.5), turned to 270 degrees
- moved D52 225.5 mm to (341.3, 42.9), turned to 90 degrees
- moved D51 219.4 mm to (330.2, 42.9), turned to 90 degrees
- moved D76 206.8 mm to (245.3, 75.4), turned to 270 degrees
- moved D14 206.5 mm to (254.0, 4.76), turned to 90 degrees
- moved D50 204.8 mm to (311.1, 42.9), turned to 90 degrees
- moved D81 204.4 mm to (341.3, 70.6), turned to 270 degrees
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Connections:
- J1 pad A4: Net-(J1-PadA4) -> VBUS
- J1 pad A6: Net-(J1-PadA6) -> D+
- J1 pad A7: Net-(J1-PadA7) -> D-
- J1 pad B4: Net-(J1-PadB4) -> VBUS
- J1 pad B6: Net-(J1-PadB6) -> D+
- J1 pad B7: Net-(J1-PadB7) -> D-
- J1 pad S: Net-(J1-PadS) -> GND
- U1 pad 32: Net-(U1-Pad32) -> D-
- U1 pad 33: Net-(U1-Pad33) -> D+
- U1 pad 34: Net-(U1-Pad34) -> SWDIO
- U1 pad 37: Net-(U1-Pad37) -> SWCLK
- U1 pad 44: Net-(U1-Pad44) -> BOOT0
- U1 pad 7: Net-(U1-Pad7) -> NRST

Commit message: routing
Parts:
- moved D2 11.3 mm to (27.2, 4.76)
- moved J2 9.53 mm to (-4.76, 38.1)
- moved CB1 4.27 mm to (14.3, 34.9)
- moved CB3 2.51 mm to (26.2, 23.8), turned to 0 degrees
- moved U1 2.51 mm to (19.1, 28.6)
- moved CB2 2.38 mm to (11.9, 24.6), turned to 180 degrees
- moved D52 1.59 mm to (339.7, 42.9)
- moved CB4 0.79 mm to (29.4, 30.2)
- moved CB5 0.79 mm to (27.0, 30.2)
Routing:
- net row0: track 0.00 -> 355.4 mm, vias 0 -> 2
- net row4: track 0.00 -> 338.8 mm
- net row1: track 0.00 -> 330.7 mm, vias 0 -> 2
- net row2: track 0.00 -> 308.1 mm
- net row3: track 0.00 -> 286.0 mm
- net col12: track 0.00 -> 92.8 mm
- net col2: track 0.00 -> 92.0 mm
- net col11: track 0.00 -> 90.0 mm
- net +3V3: track 0.00 -> 88.4 mm, vias 0 -> 5
- net col6: track 0.00 -> 87.0 mm
- net col13: track 0.00 -> 86.9 mm
- net col10: track 0.00 -> 86.1 mm
- net col14: track 0.00 -> 82.9 mm
- net col16: track 0.00 -> 76.2 mm
- net col15: track 0.00 -> 76.2 mm
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Other:
- outline, holes or cut-outs redrawn

Commit message: finished routing
Parts:
- J2: value Conn_ARM_JTAG_SWD_10 -> Conn_01x14
- moved J2 2.51 mm to (-2.38, 38.9)
- moved CRST2 0.26 mm to (33.3, 51.1)
Connections:
- U1 pad 10: Net-(U1-Pad10) -> col12
- U1 pad 11: Net-(U1-Pad11) -> col11
- U1 pad 12: Net-(U1-Pad12) -> col10
- U1 pad 13: Net-(U1-Pad13) -> col9
- U1 pad 14: Net-(U1-Pad14) -> col8
- U1 pad 15: Net-(U1-Pad15) -> col7
- U1 pad 16: Net-(U1-Pad16) -> col6
- U1 pad 17: Net-(U1-Pad17) -> col5
- U1 pad 18: Net-(U1-Pad18) -> col1
- U1 pad 19: Net-(U1-Pad19) -> col2
- U1 pad 2: Net-(U1-Pad2) -> col17
- U1 pad 20: Net-(U1-Pad20) -> col3
- U1 pad 21: Net-(U1-Pad21) -> col4
- U1 pad 22: Net-(U1-Pad22) -> col0
- U1 pad 27: Net-(U1-Pad27) -> row2
- U1 pad 28: Net-(U1-Pad28) -> row3
- U1 pad 29: Net-(U1-Pad29) -> row4
- U1 pad 3: Net-(U1-Pad3) -> col16
- U1 pad 30: Net-(U1-Pad30) -> row1
- U1 pad 31: Net-(U1-Pad31) -> row0
- U1 pad 4: Net-(U1-Pad4) -> col15
- U1 pad 5: Net-(U1-Pad5) -> col14
- U1 pad 6: Net-(U1-Pad6) -> col13
Routing:
- net col17: track 72.4 -> 403.2 mm
- net col16: track 76.2 -> 396.6 mm
- net col15: track 76.2 -> 377.4 mm
- net col14: track 82.9 -> 364.7 mm
- net col13: track 86.9 -> 332.5 mm
- net col12: track 92.8 -> 328.5 mm
- net col11: track 90.0 -> 299.4 mm
- net col10: track 86.1 -> 276.2 mm
- net col9: track 67.0 -> 236.9 mm
- net col8: track 67.0 -> 218.5 mm
- net BOOT0: track 8.68 -> 157.6 mm, vias 0 -> 2
- net col7: track 67.0 -> 200.0 mm
- net +3V3: track 88.4 -> 209.8 mm, vias 5 -> 6
- net row3: track 286.0 -> 405.0 mm, vias 0 -> 2
- net col6: track 87.0 -> 201.5 mm
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